File: pcb/equilibot.kicad_pcb (KiCad board)
At the start: 4 copper layers, 88.8 x 49.5 mm, 152 parts, among them IC1 TMC5240, IC2 TMC5240, IC3 TPS561243DRLR, IC4 TPS561243DRLR, J1 Conn_01x02_Socket, J2 USB_C_Receptacle_USB2.0_16P, J3 Conn_01x04_Pin, J4 Conn_01x04_Pin, J5 Conn_01x03_Pin, J7 Conn_01x08_Pin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

Commit message: PRODUCTION
Parts:
- added J8: Conn_01x08_Pin, Connector_PinSocket_2.54mm:PinSocket_2x04_P2.54mm_Vertical, F.Cu at (148.9, 72.7)
- C51, C52: value 1u -> 2.2u; footprint Capacitor_SMD:C_0603_1608Metric -> Capacitor_SMD:C_0805_2012Metric
- R6: value 1k -> 5.6k
- moved R22 4.20 mm to (154.1, 80.7), turned to 90 degrees
- moved R11 4.00 mm to (154.1, 77.5), turned to 90 degrees
- moved C51 3.99 mm to (112.3, 72.4), turned to 180 degrees
- moved R8 3.63 mm to (154.0, 74.0), turned to 90 degrees
- moved D34 3.08 mm to (155.7, 80.8), turned to 90 degrees
- moved D33 2.72 mm to (155.7, 77.5), turned to 90 degrees
- moved D32 2.16 mm to (155.6, 74.0), turned to 90 degrees
- moved TP1 1.87 mm to (157.7, 74.5)
- moved TP3 1.26 mm to (157.7, 76.7)
- moved TP2 0.62 mm to (157.6, 78.8)
- moved C52 0.43 mm to (115.8, 69.1)
- moved C37 0.38 mm to (117.1, 85.0)
- moved C62 0.35 mm to (126.6, 108.4)
- moved R17 0.33 mm to (114.0, 85.0)
- moved C63 0.28 mm to (143.9, 109.6)
Connections:
- U1 pad 32: /SPI_CS_IMU -> /IMU_INT2
- U1 pad 33: /IMU_INT2 -> /IMU_INT1
- U1 pad 34: /IMU_INT1 -> /SPI_CS_IMU
- U1 pad 36: unconnected-(U1-RXD0-Pad36) -> Net-(J8-Pin_4)
- U1 pad 37: unconnected-(U1-TXD0-Pad37) -> Net-(J8-Pin_3)
- U1 pad 38: unconnected-(U1-IO2-Pad38) -> Net-(J8-Pin_2)
- U1 pad 39: unconnected-(U1-IO1-Pad39) -> Net-(J8-Pin_1)
- U1 pad 5: unconnected-(U1-IO5-Pad5) -> /IO5
- U1 pad 6: unconnected-(U1-IO6-Pad6) -> /IO6
- U1 pad 7: unconnected-(U1-IO7-Pad7) -> /IO7
- U1 pad 8: unconnected-(U1-IO15-Pad8) -> /IO15
Routing:
- net GND: track 87.2 -> 137.0 mm, vias 217 -> 228
- net /IO5: track 0.00 -> 29.2 mm, vias 0 -> 1
- net /IO7: track 0.00 -> 29.1 mm, vias 0 -> 1
- net /IO6: track 0.00 -> 26.1 mm, vias 0 -> 1
- net /IO15: track 0.00 -> 26.1 mm, vias 0 -> 1
- net /3V3: track 218.7 -> 198.9 mm, vias 18 -> 16
- net Net-(J8-Pin_1): track 0.00 -> 11.1 mm
- net Net-(J8-Pin_3): track 0.00 -> 10.8 mm
- net Net-(J8-Pin_4): track 0.00 -> 8.40 mm
- net Net-(J8-Pin_2): track 0.00 -> 8.06 mm
- net /VM: track 194.0 -> 201.7 mm, vias 8 -> 17
- net /5V: track 163.8 -> 161.9 mm
- net Net-(U3-VBUS): track 25.7 -> 24.3 mm, vias 0 -> 2
- net /USB_P: track 12.8 -> 11.4 mm
- net /USB_N: track 12.8 -> 11.5 mm
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Other:
- board text added: "~BST"
