File: pcb/stepper_driver.kicad_sch (KiCad schematic)
At the start: 20 parts, among them IC1 TMC5240, J3 Conn_01x04_Pin

Commit message: routing
Parts:
- C10, C7, C8, C9: footprint Capacitor_SMD:C_0805_2012Metric -> Capacitor_SMD:C_0603_1608Metric
Changed lines of the file:
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@@
 			)
 		)
-		(property "Footprint" "Capacitor_SMD:C_0805_2012Metric"
+		(property "Footprint" "Capacitor_SMD:C_0603_1608Metric"
 			(at 146.05 48.26 0)
 			(effects
@@
 			)
 		)
-		(property "Footprint" "Capacitor_SMD:C_0805_2012Metric"
+		(property "Footprint" "Capacitor_SMD:C_0603_1608Metric"
 			(at 116.84 53.34 0)
 			(effects
@@
 			)
 		)
-		(property "Footprint" "Capacitor_SMD:C_0805_2012Metric"
+		(property "Footprint" "Capacitor_SMD:C_0603_1608Metric"
 			(at 146.05 53.34 0)
 			(effects
@@
 			)
 		)
-		(property "Footprint" "Capacitor_SMD:C_0805_2012Metric"
+		(property "Footprint" "Capacitor_SMD:C_0603_1608Metric"
 			(at 116.84 48.26 0)
 			(effects

Commit message: add jlcpcb part numbers
Parts:
- C10, C7, C8, C9: value 220p -> 470p; JLCPCB Part (none) -> C1620
- C11, C54, C56, C58, C60: JLCPCB Part (none) -> C12891
- C12, C13, C14, C62: JLCPCB Part (none) -> C21120
- C15: JLCPCB Part (none) -> C28323
- C16: JLCPCB Part (none) -> C21122
- C17: value 2.7u -> 2.2u; JLCPCB Part (none) -> C377773
- IC1: JLCPCB Part (none) -> C7494373
- J3: now not fitted
- R10: JLCPCB Part (none) -> C22797
- R9: JLCPCB Part (none) -> C23189
Changed lines of the file:
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@@
+			)
+		)
+		(property "JLCPCB Part" "C12891"
+			(at 68.58 59.69 0)
+			(effects
+				(font
+					(size 1.27 1.27)
+				)
+				(hide yes)
 			)
 		)
@@
 			)
 		)
-		(property "Value" "220p"
+		(property "Value" "470p"
 			(at 149.098 46.736 90)
 			(effects
@@
 			)
 		)
+		(property "JLCPCB Part" "C1620"
+			(at 146.05 48.26 90)
+			(effects
+				(font
+					(size 1.27 1.27)
+				)
+				(hide yes)
+			)
+		)
 		(pin "2"
 		)
@@
 			)
 		)
+		(property "JLCPCB Part" "C21120"
+			(at 36.83 76.2 0)
+			(effects
+				(font
+					(size 1.27 1.27)
+				)
+				(hide yes)
+			)
+		)
 		(pin "2"
 		)
@@
 			)
 		)
+		(property "JLCPCB Part" "C21122"
+			(at 154.94 77.47 90)
+			(effects
+				(font
+					(size 1.27 1.27)
+				)
+				(hide yes)
+			)
+		)
 		(pin "2"
 		)
@@
 			)
 		)
+		(property "JLCPCB Part" "C21120"
+			(at 101.6 59.69 0)
+			(effects
+				(font
+					(size 1.27 1.27)
+				)
+				(hide yes)
+			)
+		)
 		(pin "2"
 		)
@@
 			)
 		)
+		(property "JLCPCB Part" "C21120"
+			(at 93.98 59.69 0)
+			(effects
+				(font
+					(size 1.27 1.27)
+				)
+				(hide yes)
+			)
+		)
 		(pin "2"
 		)
@@
 			)
 		)
-		(property "Value" "220p"
+		(property "Value" "470p"
 			(at 120.396 52.324 90)
 			(effects
@@
 		(property "Description" "Unpolarized capacitor, small symbol"
 			(at 116.84 53.34 0)
+			(effects
+				(font
+					(size 1.27 1.27)
+				)
+				(hide yes)
+			)
+		)
+		(property "JLCPCB Part" "C1620"
+			(at 116.84 53.34 90)
 			(effects
 				(font
@@
 			)
 		)
-		(property "Value" "220p"
+		(property "Value" "470p"
 			(at 149.098 51.816 90)
 			(effects
@@
 		(property "Description" "Unpolarized capacitor, small symbol"
 			(at 146.05 53.34 0)
+			(effects
+				(font
+					(size 1.27 1.27)
+				)
+				(hide yes)
+			)
+		)
+		(property "JLCPCB Part" "C1620"
+			(at 146.05 53.34 90)
 			(effects
 				(font
@@
 			)
 		)
-		(property "Value" "2.7u"
+		(property "Value" "2.2u"
 			(at 127.254 111.506 0)
 			(effects
@@
 			)
 		)
+		(property "JLCPCB Part" "C377773"
+			(at 127 109.22 0)
+			(effects
+				(font
+					(size 1.27 1.27)
+				)
+				(hide yes)
+			)
+		)
 		(pin "2"
 		)
@@
 		(in_bom yes)
 		(on_board yes)
-		(dnp no)
+		(dnp yes)
 		(fields_autoplaced yes)
 		(property "Reference" "J3"
@@
 			)
 		)
+		(property "JLCPCB Part" ""
+			(at 132.08 31.75 90)
+			(effects
+				(font
+					(size 1.27 1.27)
+				)
+				(hide yes)
+			)
+		)
 		(pin "3"
 		)
@@
 				)
 				(justify left top)
+				(hide yes)
+			)
+		)
+		(property "JLCPCB Part" "C7494373"
+			(at 130.81 78.74 0)
+			(effects
+				(font
+					(size 1.27 1.27)
+				)
 				(hide yes)
 			)
@@
 			)
 		)
+		(property "JLCPCB Part" "C22797"
+			(at 121.92 107.95 0)
+			(effects
+				(font
+					(size 1.27 1.27)
+				)
+				(hide yes)
+			)
+		)
 		(pin "2"
 		)
@@
 			)
 		)
+		(property "JLCPCB Part" "C12891"
+			(at 76.2 59.69 0)
+			(effects
+				(font
+					(size 1.27 1.27)
+				)
+				(hide yes)
+			)
+		)
 		(pin "2"
 		)
@@
 			)
 		)
+		(property "JLCPCB Part" "C28323"
+			(at 148.59 72.39 90)
+			(effects
+				(font
+					(size 1.27 1.27)
+				)
+				(hide yes)
+			)
+		)
 		(pin "2"
 		)
@@
 			)
 		)
+		(property "JLCPCB Part" "C12891"
+			(at 44.45 59.69 0)
+			(effects
+				(font
+					(size 1.27 1.27)
+				)
+				(hide yes)
+			)
+		)
 		(pin "2"
 		)
@@
 			)
 		)
+		(property "JLCPCB Part" "C12891"
+			(at 53.34 59.69 0)
+			(effects
+				(font
+					(size 1.27 1.27)
+				)
+				(hide yes)
+			)
+		)
 		(pin "2"
 		)
@@
 			)
 		)
+		(property "JLCPCB Part" "C23189"
+			(at 156.21 92.71 0)
+			(effects
+				(font
+					(size 1.27 1.27)
+				)
+				(hide yes)
+			)
+		)
 		(pin "2"
 		)
@@
 			)
 		)
+		(property "JLCPCB Part" "C21120"
+			(at 87.63 59.69 0)
+			(effects
+				(font
+					(size 1.27 1.27)
+				)
+				(hide yes)
+			)
+		)
 		(pin "2"
 		)
@@
 			)
 		)
-		(property "Value" "220p"
+		(property "Value" "470p"
 			(at 120.396 47.244 90)
 			(effects
@@
 		(property "Description" "Unpolarized capacitor, small symbol"
 			(at 116.84 48.26 0)
+			(effects
+				(font
+					(size 1.27 1.27)
+				)
+				(hide yes)
+			)
+		)
+		(property "JLCPCB Part" "C1620"
+			(at 116.84 48.26 90)
 			(effects
 				(font
@@
 			(at 62.23 59.69 0)
 			(effects
+				(font
+					(size 1.27 1.27)
+				)
+				(hide yes)
+			)
+		)
+		(property "JLCPCB Part" "C12891"
+			(at 62.23 59.69 0)
+			(effects

Commit message: PRODUCTION
Other:
- moved on the sheet: C10, C11, C12, C13, C14, C15, C16, C17, C54, C56, C58, C60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
